File: PCB/tracker/tracker.kicad_pcb (KiCad board)
At the start: 2 copper layers, 58 x 57.6 mm, 20 parts, among them J1 USB_C_Receptacle_USB2.0_16P, J2 Conn_01x02, J3 DISPLAY, Q1 PMOS, U1 Wio-S3, U2 AP2112K-3.3, U3 MAX-M10S-00B, U4 QMC5883P, U5 MCP73812T-420I-OT, U6 LSM6DSV32XTR

Commit message: llm review done
Parts:
- added C4: 4.7uF, Capacitor_SMD:C_0603_1608Metric_Pad1.08x0.95mm_HandSolder, F.Cu at (85.7, 122.6)
- added C5: 4.7uF, Capacitor_SMD:C_0603_1608Metric_Pad1.08x0.95mm_HandSolder, F.Cu at (106.2, 116.4)
- added C6: 4.7uF, Capacitor_SMD:C_0603_1608Metric_Pad1.08x0.95mm_HandSolder, F.Cu at (91.2, 112.4)
- added C7: 4.7uF, Capacitor_SMD:C_0603_1608Metric_Pad1.08x0.95mm_HandSolder, F.Cu at (80.6, 109.8)
- added C8: 10uF, Capacitor_SMD:C_0603_1608Metric_Pad1.08x0.95mm_HandSolder, F.Cu at (88.8, 89.2)
- added C9: 0.1uF, Capacitor_SMD:C_0603_1608Metric_Pad1.08x0.95mm_HandSolder, F.Cu at (90.4, 89.2)
- added R10: 10k, Resistor_SMD:R_0603_1608Metric_Pad0.98x0.95mm_HandSolder, F.Cu at (88.6, 109.2)
- added R11: 10k, Resistor_SMD:R_0603_1608Metric_Pad0.98x0.95mm_HandSolder, F.Cu at (105.4, 85.4)
- added R12: 10k, Resistor_SMD:R_0603_1608Metric_Pad0.98x0.95mm_HandSolder, F.Cu at (105.4, 87.2)
- added R6: 4.7k, Capacitor_SMD:C_0603_1608Metric_Pad1.08x0.95mm_HandSolder, F.Cu at (78.2, 95.4)
- added R7: 4.7k, Capacitor_SMD:C_0603_1608Metric_Pad1.08x0.95mm_HandSolder, F.Cu at (78.2, 92.9)
- added R8: 4.7k, Capacitor_SMD:C_0603_1608Metric_Pad1.08x0.95mm_HandSolder, F.Cu at (111.8, 91.6)
- added R9: 4.7k, Capacitor_SMD:C_0603_1608Metric_Pad1.08x0.95mm_HandSolder, F.Cu at (111.8, 90.0)
- added SW1: SW_Push, Button_Switch_SMD:SW_SPST_TS-1088-xR020, F.Cu at (100.2, 87.0)
- added SW2: SW_Push, Button_Switch_SMD:SW_SPST_TS-1088-xR020, F.Cu at (100.2, 82.4)
Connections:
- U5 pad 1: CHARGE_EN -> Net-(U5-CE)
Routing:
- net 3.3V: track 105.3 -> 144.8 mm, vias 1 -> 3
- net RESET: track 0.00 -> 23.5 mm
- net BOOT: track 0.00 -> 15.3 mm, vias 0 -> 2
- net IMU_SDA: track 3.19 -> 15.5 mm
- net MAG_SCK: track 5.22 -> 15.9 mm
- net MAG_SDA: track 5.36 -> 15.2 mm
- net IMU_SCK: track 2.80 -> 9.31 mm
- net CHARGE_EN: track 5.59 -> 0.00 mm, vias 2 -> 0
- net V_BAT: track 45.5 -> 50.4 mm
- net LDO_IN: track 21.1 -> 24.0 mm
- net 5V: track 41.1 -> 43.3 mm
- net Net-(U5-CE): track 0.00 -> 1.83 mm
Other:
- board text added: "BOOT"
- board text added: "RESET"

Commit message: moved shit around
Parts:
- added C10: 0.1uF, Capacitor_SMD:C_0603_1608Metric_Pad1.08x0.95mm_HandSolder, F.Cu at (87.0, 89.2)
- added C11: 0.1uF, Capacitor_SMD:C_0603_1608Metric_Pad1.08x0.95mm_HandSolder, F.Cu at (117.0, 95.2)
- added C12: 0.1uF, Capacitor_SMD:C_0603_1608Metric_Pad1.08x0.95mm_HandSolder, F.Cu at (117.0, 93.6)
- added H1: MountingHole, MountingHole:MountingHole_3.2mm_M3, F.Cu at (83.0, 85.0)
- added H2: MountingHole, MountingHole:MountingHole_3.2mm_M3, F.Cu at (115.0, 115.0)
- added H3: MountingHole, MountingHole:MountingHole_3.2mm_M3, F.Cu at (78.0, 114.0)
- added H4: MountingHole, MountingHole:MountingHole_3.2mm_M3, F.Cu at (115.0, 85.0)
- moved J2 15.5 mm to (114.8, 80.4), turned to 90 degrees
- turned C6 to 0 degrees
Connections:
- U6 pad 2: unconnected-(U6-SDx/AH1/Qvar1-Pad2) -> GND
- U6 pad 3: unconnected-(U6-SCx/AH2/Qvar2-Pad3) -> GND
Routing:
- net V_BAT: track 50.4 -> 62.9 mm
- net 3.3V: track 144.8 -> 152.8 mm
- net 5V: track 43.3 -> 47.0 mm
- net GND: track 7.03 -> 9.08 mm, vias 54 -> 53
- net IMU_SDA: track 15.5 -> 16.8 mm
- net BOOT: track 15.3 -> 16.0 mm
