File: PCB/tracker/tracker.kicad_sch (KiCad schematic)
At the start: 20 parts, among them J1 USB_C_Receptacle_USB2.0_16P, J2 Conn_01x02, J3 DISPLAY, Q1 PMOS, U1 Wio-S3, U2 AP2112K-3.3, U3 MAX-M10S-00B, U4 QMC5883P, U5 MCP73812T-420I-OT, U6 LSM6DSV32XTR

Commit message: llm review done
Parts:
- added C4, C5, C6, C7: 4.7uF, Capacitor_SMD:C_0603_1608Metric_Pad1.08x0.95mm_HandSolder, symbol Device:C_Small
- added C8: 10uF, Capacitor_SMD:C_0603_1608Metric_Pad1.08x0.95mm_HandSolder, symbol Device:C_Small
- added C9: 0.1uF, Capacitor_SMD:C_0603_1608Metric_Pad1.08x0.95mm_HandSolder, symbol Device:C_Small
- added R10, R11, R12: 10k, Resistor_SMD:R_0603_1608Metric_Pad0.98x0.95mm_HandSolder, symbol Device:R_Small
- added R6, R7, R8, R9: 4.7k, Capacitor_SMD:C_0603_1608Metric_Pad1.08x0.95mm_HandSolder, symbol Device:R_Small
- added SW1, SW2: SW_Push, Button_Switch_SMD:SW_SPST_TS-1088-xR020, symbol Switch:SW_Push
Connections:
- net 3.3V: now also C5.1, C8.1, C9.2, R11.1, R12.2, R6.2, R7.2, R8.2, R9.2
- net 5V: now also C6.1, R10.1
- net BOOT: now also R12.1, SW1.1
- net CHARGE_EN: no longer U5.1 (CE)
- net GND: now also C4.2, C5.2, C6.2, C7.2, C8.2, C9.1, SW1.2, SW2.2
- net IMU_SCK: now also R8.1
- net IMU_SDA: now also R9.1
- net LDO_IN: now also C4.1
- net MAG_SCK: now also R7.1
- net MAG_SDA: now also R6.1
- net RESET: now also R11.2, SW2.1
- net V_BAT: now also C7.1
- new net: R10.2, U5.1 (CE)
Other:
- moved on the sheet: J3, U2

Commit message: moved shit around
Parts:
- added C10, C11, C12: 0.1uF, Capacitor_SMD:C_0603_1608Metric_Pad1.08x0.95mm_HandSolder, symbol Device:C_Small
- added H1, H2, H3, H4: MountingHole, MountingHole:MountingHole_3.2mm_M3, symbol Mechanical:MountingHole
Connections:
- net 3.3V: now also C10.2, C11.2, C12.2
- net GND: now also U6.2 (SDx/AH1/Qvar1), U6.3 (SCx/AH2/Qvar2), C10.1, C11.1, C12.1
- no-connect marks 35 -> 33

Commit message: ahhhh
Parts:
- D1: footprint Diode_SMD:D_SMA-SMB_Universal_Handsoldering -> Diode_SMD:D_SOD-123F
- R6, R7, R8, R9: footprint Capacitor_SMD:C_0603_1608Metric_Pad1.08x0.95mm_HandSolder -> Resistor_SMD:R_0603_1608Metric_Pad0.98x0.95mm_HandSolder
Changed lines of the file:
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@@
 			)
 		)
-		(property "Footprint" "Capacitor_SMD:C_0603_1608Metric_Pad1.08x0.95mm_HandSolder"
+		(property "Footprint" "Resistor_SMD:R_0603_1608Metric_Pad0.98x0.95mm_HandSolder"
 			(at 262.89 143.51 0)
 			(hide yes)
@@
 			)
 		)
-		(property "Footprint" "Capacitor_SMD:C_0603_1608Metric_Pad1.08x0.95mm_HandSolder"
+		(property "Footprint" "Resistor_SMD:R_0603_1608Metric_Pad0.98x0.95mm_HandSolder"
 			(at 262.89 151.13 0)
 			(hide yes)
@@
 			)
 		)
-		(property "Footprint" "Capacitor_SMD:C_0603_1608Metric_Pad1.08x0.95mm_HandSolder"
+		(property "Footprint" "Resistor_SMD:R_0603_1608Metric_Pad0.98x0.95mm_HandSolder"
 			(at 262.89 135.89 0)
 			(hide yes)
@@
 			)
 		)
-		(property "Footprint" "Capacitor_SMD:C_0603_1608Metric_Pad1.08x0.95mm_HandSolder"
+		(property "Footprint" "Resistor_SMD:R_0603_1608Metric_Pad0.98x0.95mm_HandSolder"
 			(at 262.89 128.27 0)
 			(hide yes)
@@
 			)
 		)
-		(property "Footprint" "Diode_SMD:D_SMA-SMB_Universal_Handsoldering"
+		(property "Footprint" "Diode_SMD:D_SOD-123F"
 			(at 175.26 21.59 0)
 			(hide yes)
